Commit message: correct the point cloud color, add necessary link for point cloud frame

File: rover_descriptions/zhurong_description/urdf/sensor_obstacle_stereo_camera.xacro (robot description, xacro)
@@ -116,4 +116,10 @@
       <origin xyz="0.012 0 0.015" rpy="0 0 0"/>
     </joint>
+    <link name="camera_obs_F_optical_frame"/>
+    <joint name="camera_obs_F_optical_joint" type="fixed">
+      <parent link="camera_obs_F_link"/>
+      <child link="camera_obs_F_optical_frame"/>
+      <origin xyz="0 0 0" rpy="-1.57 0 -1.57"/>
+    </joint>
     <link name="obsZEDSupport_B_Link">
       <inertial>
@@ -229,4 +235,10 @@
       <origin xyz="0.012 0 0.015" rpy="0 0 0"/>
     </joint>
+    <link name="camera_obs_B_optical_frame"/>
+    <joint name="camera_obs_B_optical_joint" type="fixed">
+      <parent link="camera_obs_B_link"/>
+      <child link="camera_obs_B_optical_frame"/>
+      <origin xyz="0 0 0" rpy="-1.57 0 -1.57"/>
+    </joint>
   </xacro:macro>
 </robot>

File: rover_descriptions/zhurong_description/urdf/sensor_stereo_camera2.xacro (robot description, xacro)
@@ -292,9 +292,9 @@
 			<origin xyz="-10 0 10" rpy="0 0.5 0"/>
 		</joint> -->
-		<link name="camera_nav_pointcloud_link"/>
+		<link name="camera_nav_optical_frame"/>
 		<joint name="camera_nav_pointcloud_joint" type="fixed">
 			<origin xyz="0 0 0" rpy="-1.57 0 -1.57"/>
 			<parent link="camera_nav_link"/>
-			<child link="camera_nav_pointcloud_link"/>
+			<child link="camera_nav_optical_frame"/>
 		</joint>
 	</xacro:macro>
