Commit message: update version

File: rover_descriptions/zhurong_description/urdf/chassis.xacro (robot description, xacro)
@@ -2,10 +2,4 @@
 <robot xmlns:xacro="http://www.ros.org/wiki/xacro">
 	<xacro:macro name="chassis_body" params="">
-		<!-- <link name='world'/>
-		<joint name="world_joint" type="floating">
-				<parent link="world"/>
-				<child link="chassis"/>
-				<origin xyz="0 0 0" rpy="0 0 0"/>
-		</joint> -->
 		<link name='chassis'>
 			<collision>
@@ -24,7 +18,7 @@
 					<mesh filename="package://zhurong_description/meshes/base_link.STL" />
 				</geometry>
-				<!-- <material name="">
-						<color rgba="0.79216 0.81961 0.93333 1" />
-				</material> -->
+				<material name="">
+						<color rgba="0.51 0.38 0.15 1" />
+				</material>
 			</visual>
 			<inertial>
@@ -57,4 +51,10 @@
 			</visual>
 		</gazebo>
+		<link name="imu_link"/>
+		<joint name="imu_joint" type="fixed">
+				<parent link="chassis"/>
+				<child link="imu_link"/>
+				<origin xyz="0.0 0 0" rpy="0 0 0"/>
+		</joint>
 		<!-- Used for fixing robot to Gazebo 'chassis' -->
 		<link name="nav_base_link" >

File: rover_descriptions/zhurong_description/urdf/sensor_roLIDAR.xacro (robot description, xacro)
@@ -71,5 +71,5 @@
 				</geometry>
 				<material name="">
-					<color rgba="1 0.592156862745098 1 1" />
+					<color rgba="1 1 1 1" />
 				</material>
 			</visual>

File: rover_descriptions/zhurong_description/urdf/sensor_stereo_camera2.xacro (robot description, xacro)
@@ -137,5 +137,5 @@
 			</visual>
 		</gazebo>
-		<joint name="PTZYaw_joint" type="fixed">
+		<joint name="PTZYaw_joint" type="revolute">
 			<origin xyz="0 0 0.023"
 							rpy="0 0 0" />
@@ -147,5 +147,5 @@
 			<!-- <safety_controller soft_upper="2" soft_lower="1" k_position="1" k_velocity="2" /> -->
 		</joint>
-		<!-- <transmission name="PTZYaw_trans">
+		<transmission name="PTZYaw_trans">
 			<type>transmission_interface/SimpleTransmission</type>
 			<joint name="PTZYaw_joint">
@@ -156,5 +156,5 @@
 				<mechanicalReduction>1</mechanicalReduction>
 			</actuator>
-		</transmission> -->
+		</transmission>
 		<link name="PTZPitch_Link">
 			<inertial>
@@ -199,7 +199,8 @@
 			</visual>
 		</gazebo>
-		<joint name="PTZPitch_joint" type="fixed">
+		<joint name="PTZPitch_joint" type="revolute">
+		<!-- 0.63 -->
 			<origin xyz="0 0.055 0.062"
-							rpy="0 0.63 0" />
+							rpy="0 0.5 0" />
 			<parent link="PTZYaw_Link" />
 			<child link="PTZPitch_Link" />
@@ -209,5 +210,5 @@
 			<!-- <safety_controller soft_upper="2" soft_lower="1" k_position="1" k_velocity="2" /> -->
 		</joint>
-		<!-- <transmission name="PTZPitch_trans">
+		<transmission name="PTZPitch_trans">
 			<type>transmission_interface/SimpleTransmission</type>
 			<joint name="PTZPitch_joint">
@@ -218,5 +219,5 @@
 				<mechanicalReduction>1</mechanicalReduction>
 			</actuator>
-		</transmission> -->
+		</transmission>
 		<link name='ZEDNav_Link'>
 			<collision>
@@ -284,6 +285,5 @@
 			<origin xyz="0.03 0 -0." rpy="0 0 0"/>
 		</joint>
-		<link name="gald_camera">
-		<!-- <pose>0 0 10 0 0 0</pose> -->
+		<!-- <link name="gald_camera">
 		</link>
 		<joint name="camera_sky_joint" type="fixed">
@@ -291,4 +291,10 @@
 			<child link="gald_camera"/>
 			<origin xyz="-10 0 10" rpy="0 0.5 0"/>
+		</joint> -->
+		<link name="camera_nav_pointcloud_link"/>
+		<joint name="camera_nav_pointcloud_joint" type="fixed">
+			<origin xyz="0 0 0" rpy="-1.57 0 -1.57"/>
+			<parent link="camera_nav_link"/>
+			<child link="camera_nav_pointcloud_link"/>
 		</joint>
 	</xacro:macro>

File: rover_descriptions/zhurong_description/urdf/wheel.xacro (robot description, xacro)
@@ -17,4 +17,7 @@
 						<mesh filename="package://zhurong_description/meshes/wheel_LB_Link.STL"/>
 					</geometry>
+					<material name="">
+						<color rgba="0.53 0.51 0.49 1" />
+					</material>
 				</visual>
 				<inertial>
@@ -73,5 +76,5 @@
 			</transmission>
 			<gazebo>
-				<plugin name="${wheel_name}_terrain_interaction" filename="libTerramechanicsPlugin.so">
+				<plugin name="${wheel_name}_terrain_interaction" filename="${PLUGINS['$(arg Plugin)']}">
 					<base_link>${wheel_conector_name}</base_link>
 					<wheel_link>${wheel_name}</wheel_link>
@@ -80,5 +83,5 @@
 					<wheel_r>0.15</wheel_r>
 					<wheel_b>0.2</wheel_b>
-					<wheel_h>0.00</wheel_h>
+					<wheel_h>0.01</wheel_h>
 					<FN_AVE>250</FN_AVE>
 				</plugin>

File: rover_descriptions/zhurong_description/urdf/zhurong_mars_rover.xacro (robot description, xacro)
@@ -14,5 +14,5 @@
 	<xacro:include filename="$(find zhurong_description)/urdf/right_wheel_group.xacro" />
 	<!-- Sensor Mast -->
-	<xacro:include filename="$(find zhurong_description)/urdf/sensor_stereo_camera.xacro" />
+	<xacro:include filename="$(find zhurong_description)/urdf/sensor_stereo_camera2.xacro" />
 	<xacro:include filename="$(find zhurong_description)/urdf/sensor_LIDAR_group.xacro" />
 	<xacro:include filename="$(find zhurong_description)/urdf/sensor_obstacle_stereo_camera.xacro" />

File: rover_descriptions/zhurong_description/urdf/zhurong_mars_rover_properties.xacro (robot description, xacro)
@@ -61,3 +61,6 @@
 	<xacro:property name="PTZPitch_Mass" value="0.0640993648047983"/>
 	<xacro:property name="ZEDNav_Mass" value="0.3"/>
+	<xacro:property name="YAML_FILE" value="$(find rover_gazebo_plugins)/config/TerramechanicsPluginParam.yaml" />
+	<xacro:property name="PLUGINS" value="${load_yaml(YAML_FILE)}"/>
+	<xacro:arg name="Plugin" default="Plugin" />
 </robot>

File: rover_gazebo/urdf/zhurong_gazebo.xacro (robot description, xacro)
@@ -14,5 +14,5 @@
 	<xacro:include filename="$(find zhurong_description)/urdf/right_wheel_group.xacro" />
 	<!-- Sensor Mast -->
-	<xacro:include filename="$(find zhurong_description)/urdf/sensor_stereo_camera.xacro" />
+	<xacro:include filename="$(find zhurong_description)/urdf/sensor_stereo_camera2.xacro" />
 	<xacro:include filename="$(find zhurong_description)/urdf/sensor_LIDAR_group.xacro" />
 	<xacro:include filename="$(find zhurong_description)/urdf/sensor_obstacle_stereo_camera.xacro" />

Commit message: neotic first commit

File: rover_descriptions/zhurong_description/urdf/chassis.xacro (robot description, xacro)
@@ -2,4 +2,10 @@
 <robot xmlns:xacro="http://www.ros.org/wiki/xacro">
 	<xacro:macro name="chassis_body" params="">
+		<link name = 'base_link'/>
+		<joint name="base_c_joint" type="fixed">
+				<parent link="base_link"/>
+				<child link="chassis"/>
+				<origin xyz="0.0 0 0" rpy="0 0 0"/>
+		</joint>
 		<link name='chassis'>
 			<collision>

File: rover_descriptions/zhurong_description/urdf/left_wheel_group.xacro (robot description, xacro)
@@ -203,5 +203,5 @@
 			</actuator>
 		</transmission>
-		<wheel
+		<xacro:wheel
 			wheel_name="front_wheel_L"
 			wheel_conector_name="suspension_steer_F_L"
@@ -258,5 +258,5 @@
 			</actuator>
 		</transmission>
-		<wheel
+		<xacro:wheel
 			wheel_name="middle_wheel_L"
 			wheel_conector_name="suspension_steer_M_L"
@@ -313,5 +313,5 @@
 			</actuator>
 		</transmission>
-		<wheel
+		<xacro:wheel
 			wheel_name="back_wheel_L"
 			wheel_conector_name="suspension_steer_B_L"

File: rover_descriptions/zhurong_description/urdf/right_wheel_group.xacro (robot description, xacro)
@@ -203,5 +203,5 @@
 			</actuator>
 		</transmission>
-		<wheel
+		<xacro:wheel
 			wheel_name="front_wheel_R"
 			wheel_conector_name="suspension_steer_F_R"
@@ -258,5 +258,5 @@
 			</actuator>
 		</transmission>
-		<wheel
+		<xacro:wheel
 			wheel_name="middle_wheel_R"
 			wheel_conector_name="suspension_steer_M_R"
@@ -313,5 +313,5 @@
 			</actuator>
 		</transmission>
-		<wheel
+		<xacro:wheel
 			wheel_name="back_wheel_R"
 			wheel_conector_name="suspension_steer_B_R"

File: rover_gazebo/urdf/zhurong_gazebo.xacro (robot description, xacro)
@@ -18,10 +18,10 @@
 	<xacro:include filename="$(find zhurong_description)/urdf/sensor_obstacle_stereo_camera.xacro" />
 	<xacro:include filename="$(find zhurong_description)/urdf/sensor_roLIDAR.xacro" />
-	<chassis_body/>
-	<left_wheel_tree/>
-	<right_wheel_tree/>
-	<sensor_ZEDNav/>
-	<sensor_LIDAR/>
-	<sensor_obsZED/>
-	<sensor_roLIDAR/>
+	<xacro:chassis_body/>
+	<xacro:left_wheel_tree/>
+	<xacro:right_wheel_tree/>
+	<xacro:sensor_ZEDNav/>
+	<xacro:sensor_LIDAR/>
+	<xacro:sensor_obsZED/>
+	<xacro:sensor_roLIDAR/>
 </robot>

Commit message: change the collision check of the body to mesh, rather than the manually box

File: rover_descriptions/zhurong_description/urdf/chassis.xacro (robot description, xacro)
@@ -10,10 +10,13 @@
 		<link name='chassis'>
 			<collision>
-				<origin xyz="0.85 0 0.105"
+				<!-- <origin xyz="0.85 0 0.105"
+								rpy="0 0 0"/> -->
+				<origin xyz="0 0 0"
 								rpy="0 0 0"/>
 				<geometry>
+					<mesh filename="package://zhurong_description/meshes/base_link.STL" />
 					<!-- <box size="1.252 0.832 0.502"/> -->
 					<!-- <box size="1.8 1.6 0.502"/> -->
-					<box size="0.25 1.6 0.502"/>
+					<!-- <box size="0.25 1.6 0.502"/> -->
 				</geometry>
 			</collision>
@@ -65,5 +68,5 @@
 		<!-- Used for fixing robot to Gazebo 'chassis' -->
 		<link name="nav_base_link" >
-			<collision>
+			<!-- <collision>
 				<origin xyz="-0.3 0 0.105"
 								rpy="0 0 0"/>
@@ -71,5 +74,5 @@
 					<box size="1.5 1.6 0.502"/>
 				</geometry>
-			</collision>
+			</collision> -->
 		</link>
 		<joint name="base_joint" type="fixed">

Commit message: renewed version

File: rover_descriptions/zhurong_description/urdf/chassis.xacro (robot description, xacro)
@@ -2,4 +2,10 @@
 <robot xmlns:xacro="http://www.ros.org/wiki/xacro">
 	<xacro:macro name="chassis_body" params="">
+		<link name = 'base_link'/>
+		<joint name="base_c_joint" type="fixed">
+				<parent link="base_link"/>
+				<child link="chassis"/>
+				<origin xyz="0.0 0 0" rpy="0 0 0"/>
+		</joint>
 		<link name='chassis'>
 			<collision>
@@ -70,5 +76,6 @@
 				<parent link="chassis"/>
 				<child link="nav_base_link"/>
-				<origin xyz="0.2 0 0" rpy="0 0 0"/>
+				<origin xyz="0 0 0" rpy="0 0 0"/>
+				<!-- <origin xyz="0.2 0 0" rpy="0 0 0"/> -->
 		</joint>
 	</xacro:macro>

File: rover_descriptions/zhurong_description/urdf/left_wheel_group.xacro (robot description, xacro)
@@ -203,5 +203,5 @@
 			</actuator>
 		</transmission>
-		<wheel
+		<xacro:wheel
 			wheel_name="front_wheel_L"
 			wheel_conector_name="suspension_steer_F_L"
@@ -258,5 +258,5 @@
 			</actuator>
 		</transmission>
-		<wheel
+		<xacro:wheel
 			wheel_name="middle_wheel_L"
 			wheel_conector_name="suspension_steer_M_L"
@@ -313,5 +313,5 @@
 			</actuator>
 		</transmission>
-		<wheel
+	<xacro:wheel
 			wheel_name="back_wheel_L"
 			wheel_conector_name="suspension_steer_B_L"

File: rover_descriptions/zhurong_description/urdf/right_wheel_group.xacro (robot description, xacro)
@@ -203,5 +203,5 @@
 			</actuator>
 		</transmission>
-		<wheel
+	<xacro:wheel
 			wheel_name="front_wheel_R"
 			wheel_conector_name="suspension_steer_F_R"
@@ -258,5 +258,5 @@
 			</actuator>
 		</transmission>
-		<wheel
+	<xacro:wheel
 			wheel_name="middle_wheel_R"
 			wheel_conector_name="suspension_steer_M_R"
@@ -313,5 +313,5 @@
 			</actuator>
 		</transmission>
-		<wheel
+	<xacro:wheel
 			wheel_name="back_wheel_R"
 			wheel_conector_name="suspension_steer_B_R"

File: rover_descriptions/zhurong_description/urdf/sensor_obstacle_stereo_camera.xacro (robot description, xacro)
@@ -92,5 +92,5 @@
       <origin
         xyz="0.035358 0 -0.036993"
-        rpy="0 0.7 0" />
+        rpy="0 0.4 0" />
       <parent link="obsZEDSupport_F_Link" />
       <child link="obsZED_F_Link" />
@@ -205,5 +205,5 @@
       <origin
         xyz="0.035358 0 -0.036993"
-        rpy="0 0.92502 0" />
+        rpy="0 0.4 0" />
       <parent link="obsZEDSupport_B_Link" />
       <child link="obsZED_B_Link" />
@@ -229,4 +229,28 @@
       <origin xyz="0.012 0 0.015" rpy="0 0 0"/>
     </joint>
+    <link name="camera_obs_F_pointcloud_link"/>
+		<joint name="camera_obs_F_pointcloud_joint" type="fixed">
+			<origin xyz="0 0 0" rpy="-1.57 0 -1.57"/>
+			<parent link="camera_obs_F_link"/>
+			<child link="camera_obs_F_pointcloud_link"/>
+		</joint>
+    <link name="camera_obs_B_pointcloud_link"/>
+    <joint name="camera_obs_B_pointcloud_joint" type="fixed">
+      <origin xyz="0 0 0" rpy="-1.57 0 -1.57"/>
+      <parent link="camera_obs_B_link"/>
+      <child link="camera_obs_B_pointcloud_link"/>
+    </joint>
+    <link name="camera_obs_L_pointcloud_link"/>
+    <joint name="camera_obs_L_pointcloud_joint" type="fixed">
+      <origin xyz="0 0 0" rpy="-1.57 0 -1.57"/>
+      <parent link="camera_obs_L_link"/>
+      <child link="camera_obs_L_pointcloud_link"/>
+    </joint>
+    <link name="camera_obs_R_pointcloud_link"/>
+    <joint name="camera_obs_R_pointcloud_joint" type="fixed">
+      <origin xyz="0 0 0" rpy="-1.57 0 -1.57"/>
+      <parent link="camera_obs_R_link"/>
+      <child link="camera_obs_R_pointcloud_link"/>
+    </joint>
   </xacro:macro>
 </robot>

File: rover_descriptions/zhurong_description/urdf/wheel.xacro (robot description, xacro)
@@ -39,10 +39,10 @@
 			</link>
 			<gazebo reference="${wheel_name}">
-				<mu1 value="1.0"/>
-				<mu2 value="1.0"/>
-				<kp  value="10000000.0" />
-				<kd>100.0</kd>
-				<minDepth>0.001</minDepth>
-				<maxVel>1.0</maxVel>
+				<mu1 value="0.0"/>
+				<mu2 value="0.0"/>
+				<kp  value="0.0" />
+				<kd>0.0</kd>
+				<minDepth>0.0</minDepth>
+				<maxVel>0.0</maxVel>
 				<!--kd  value="1.0" />
 				<fdir1 value="1 0 0"/-->

File: rover_descriptions/zhurong_description/urdf/zhurong_mars_rover.xacro (robot description, xacro)
@@ -17,4 +17,5 @@
 	<xacro:include filename="$(find zhurong_description)/urdf/sensor_LIDAR_group.xacro" />
 	<xacro:include filename="$(find zhurong_description)/urdf/sensor_obstacle_stereo_camera.xacro" />
+	<xacro:include filename="$(find zhurong_description)/urdf/sensor_obstacle_side_camera.xacro" />
 	<xacro:include filename="$(find zhurong_description)/urdf/sensor_roLIDAR.xacro" />
 	<chassis_body/>
@@ -24,4 +25,5 @@
 	<sensor_LIDAR/>
 	<sensor_obsZED/>
+	<sensor_obsZED_side/>
 	<sensor_roLIDAR/>
 </robot>

File: rover_gazebo/urdf/zhurong_gazebo.xacro (robot description, xacro)
@@ -17,11 +17,15 @@
 	<xacro:include filename="$(find zhurong_description)/urdf/sensor_LIDAR_group.xacro" />
 	<xacro:include filename="$(find zhurong_description)/urdf/sensor_obstacle_stereo_camera.xacro" />
+	<xacro:include filename="$(find zhurong_description)/urdf/sensor_obstacle_side_camera.xacro" />
 	<xacro:include filename="$(find zhurong_description)/urdf/sensor_roLIDAR.xacro" />
-	<chassis_body/>
-	<left_wheel_tree/>
-	<right_wheel_tree/>
-	<sensor_ZEDNav/>
-	<sensor_LIDAR/>
-	<sensor_obsZED/>
-	<sensor_roLIDAR/>
+	<xacro:include filename="$(find zhurong_description)/urdf/sensor_VLP16.xacro"/>
+	<!-- <xacro:include filename="$(find zhurong_description)/urdf/sensor_HDL32E.xacro"/> -->
+	<xacro:chassis_body/>
+	<xacro:left_wheel_tree/>
+	<xacro:right_wheel_tree/>
+	<xacro:sensor_ZEDNav/>
+	<xacro:sensor_LIDAR/>
+	<xacro:sensor_obsZED/>
+	<xacro:sensor_obsZED_side/>
+	<xacro:sensor_roLIDAR/>
 </robot>
